Commit message: working ompl planning through rviz for argallab robot
need to fix multiple robot state publishers
need to fix velocity limits, now too low

File: ada_hardware/urdf/argallab_hardware.ros2_control.xacro (robot description, xacro)
@@ -1,5 +1,5 @@
 <?xml version="1.0"?>
 <robot xmlns:xacro="http://www.ros.org/wiki/xacro">
-  <xacro:macro name="ada_hardware_interface" params="name prefix:=j2n6s200 sim">
+  <xacro:macro name="ada_hardware_interface" params="name prefix:=j2s7s300 sim:=none">
     <ros2_control name="${name}" type="system">
       <hardware>
@@ -66,4 +66,13 @@
         <state_interface name="effort"/>
       </joint>
+      <!-- Added this to include 7th joint for 7 DOF robot -->
+      <joint name="${prefix}_joint_7">
+        <command_interface name="position"/>
+        <command_interface name="velocity"/>
+        <command_interface name="effort"/>
+        <state_interface name="position"/>
+        <state_interface name="velocity"/>
+        <state_interface name="effort"/>
+      </joint>
       <!-- Finger DOFs -->
       <joint name="${prefix}_joint_finger_1">
@@ -83,4 +92,13 @@
         <state_interface name="effort"/>
       </joint>
+      <!-- Added this to include 3rd jaco finger for 7 DOF robot -->
+      <joint name="${prefix}_joint_finger_3">
+        <command_interface name="position"/>
+        <command_interface name="velocity"/>
+        <command_interface name="effort"/>
+        <state_interface name="position"/>
+        <state_interface name="velocity"/>
+        <state_interface name="effort"/>
+      </joint>
     </ros2_control>
   </xacro:macro>

File: ada_hardware/urdf/argallab_hardware.xacro (robot description, xacro)
@@ -1,9 +1,11 @@
 <?xml version="1.0"?>
 <!-- j2n6s200 refers to jaco v2 6DOF non-spherical 2fingers -->
+<!-- j2s7s300 refers to jaco v2 7DOF 3 fingers robot -->
 <robot xmlns:xi="http://www.w3.org/2001/XInclude"
 	xmlns:xacro="http://www.ros.org/wiki/xacro" name="ada_hardware">
   <xacro:arg name="sim" default="none" />
-  <xacro:include filename="$(find ada_description)/urdf/ada.xacro"/>
-  <xacro:include filename="$(find ada_hardware)/urdf/ada_hardware.ros2_control.xacro"/>
+  <xacro:include filename="$(find ada_description)/urdf/argallab_jaco.xacro"/>
+  <!-- above used to be ada.xacro -->
+  <xacro:include filename="$(find ada_hardware)/urdf/argallab_hardware.ros2_control.xacro"/>
   <xacro:ada_hardware_interface
     name="Jaco2"

File: ada_moveit/config/argallab_jaco.ros2_control.xacro (robot description, xacro)
@@ -1,5 +1,5 @@
 <?xml version="1.0"?>
 <robot xmlns:xacro="http://www.ros.org/wiki/xacro">
-    <xacro:macro name="ada_ros2_control" params="name initial_positions_file sim">
+    <xacro:macro name="argallab_jaco_ros2_control" params="name initial_positions_file sim">
         <xacro:property name="initial_positions" value="${xacro.load_yaml(initial_positions_file)['initial_positions']}"/>
         <ros2_control name="${name}" type="system">
@@ -18,10 +18,10 @@
                 </xacro:if>
               </hardware>
-            <joint name="j2n6s200_joint_1">
+            <joint name="j2s7s300_joint_1">
                 <command_interface name="position"/>
                 <command_interface name="velocity"/>
                 <command_interface name="effort"/>
                 <state_interface name="position">
-                  <param name="initial_value">${initial_positions['j2n6s200_joint_1']}</param>
+                  <param name="initial_value">${initial_positions['j2s7s300_joint_1']}</param>
                 </state_interface>
                 <state_interface name="velocity">
@@ -32,10 +32,10 @@
                 </state_interface>
             </joint>
-            <joint name="j2n6s200_joint_2">
+            <joint name="j2s7s300_joint_2">
                 <command_interface name="position"/>
                 <command_interface name="velocity"/>
                 <command_interface name="effort"/>
                 <state_interface name="position">
-                  <param name="initial_value">${initial_positions['j2n6s200_joint_2']}</param>
+                  <param name="initial_value">${initial_positions['j2s7s300_joint_2']}</param>
                 </state_interface>
                 <state_interface name="velocity">
@@ -46,10 +46,10 @@
                 </state_interface>
             </joint>
-            <joint name="j2n6s200_joint_3">
+            <joint name="j2s7s300_joint_3">
                 <command_interface name="position"/>
                 <command_interface name="velocity"/>
                 <command_interface name="effort"/>
                 <state_interface name="position">
-                  <param name="initial_value">${initial_positions['j2n6s200_joint_3']}</param>
+                  <param name="initial_value">${initial_positions['j2s7s300_joint_3']}</param>
                 </state_interface>
                 <state_interface name="velocity">
@@ -60,10 +60,10 @@
                 </state_interface>
             </joint>
-            <joint name="j2n6s200_joint_4">
+            <joint name="j2s7s300_joint_4">
                 <command_interface name="position"/>
                 <command_interface name="velocity"/>
                 <command_interface name="effort"/>
                 <state_interface name="position">
-                  <param name="initial_value">${initial_positions['j2n6s200_joint_4']}</param>
+                  <param name="initial_value">${initial_positions['j2s7s300_joint_4']}</param>
                 </state_interface>
                 <state_interface name="velocity">
@@ -74,10 +74,10 @@
                 </state_interface>
             </joint>
-            <joint name="j2n6s200_joint_5">
+            <joint name="j2s7s300_joint_5">
                 <command_interface name="position"/>
                 <command_interface name="velocity"/>
                 <command_interface name="effort"/>
                 <state_interface name="position">
-                  <param name="initial_value">${initial_positions['j2n6s200_joint_5']}</param>
+                  <param name="initial_value">${initial_positions['j2s7s300_joint_5']}</param>
                 </state_interface>
                 <state_interface name="velocity">
@@ -88,10 +88,10 @@
                 </state_interface>
             </joint>
-            <joint name="j2n6s200_joint_6">
+            <joint name="j2s7s300_joint_6">
                 <command_interface name="position"/>
                 <command_interface name="velocity"/>
                 <command_interface name="effort"/>
                 <state_interface name="position">
-                  <param name="initial_value">${initial_positions['j2n6s200_joint_6']}</param>
+                  <param name="initial_value">${initial_positions['j2s7s300_joint_6']}</param>
                 </state_interface>
                 <state_interface name="velocity">
@@ -102,10 +102,10 @@
                 </state_interface>
             </joint>
-            <joint name="j2n6s200_joint_finger_1">
+            <joint name="j2s7s300_joint_7">
                 <command_interface name="position"/>
                 <command_interface name="velocity"/>
                 <command_interface name="effort"/>
                 <state_interface name="position">
-                  <param name="initial_value">${initial_positions['j2n6s200_joint_finger_1']}</param>
+                  <param name="initial_value">${initial_positions['j2s7s300_joint_7']}</param>
                 </state_interface>
                 <state_interface name="velocity">
@@ -116,10 +116,38 @@
                 </state_interface>
             </joint>
-            <joint name="j2n6s200_joint_finger_2">
+            <joint name="j2s7s300_joint_finger_1">
                 <command_interface name="position"/>
                 <command_interface name="velocity"/>
                 <command_interface name="effort"/>
                 <state_interface name="position">
-                  <param name="initial_value">${initial_positions['j2n6s200_joint_finger_2']}</param>
+                  <param name="initial_value">${initial_positions['j2s7s300_joint_finger_1']}</param>
+                </state_interface>
+                <state_interface name="velocity">
+                    <param name="initial_value">0.0</param>
+                </state_interface>
+                <state_interface name="effort">
+                    <param name="initial_value">0.0</param>
+                </state_interface>
+            </joint>
+            <joint name="j2s7s300_joint_finger_2">
+                <command_interface name="position"/>
+                <command_interface name="velocity"/>
+                <command_interface name="effort"/>
+                <state_interface name="position">
+                  <param name="initial_value">${initial_positions['j2s7s300_joint_finger_2']}</param>
+                </state_interface>
+                <state_interface name="velocity">
+                    <param name="initial_value">0.0</param>
+                </state_interface>
+                <state_interface name="effort">
+                    <param name="initial_value">0.0</param>
+                </state_interface>
+            </joint>
+            <joint name="j2s7s300_joint_finger_3">
+                <command_interface name="position"/>
+                <command_interface name="velocity"/>
+                <command_interface name="effort"/>
+                <state_interface name="position">
+                  <param name="initial_value">${initial_positions['j2s7s300_joint_finger_3']}</param>
                 </state_interface>
                 <state_interface name="velocity">

File: ada_moveit/config/argallab_jaco.urdf.xacro (robot description, xacro)
@@ -1,11 +1,11 @@
 <?xml version="1.0"?>
-<robot xmlns:xacro="http://www.ros.org/wiki/xacro" name="ada">
+<robot xmlns:xacro="http://www.ros.org/wiki/xacro" name="argallab_jaco">
     <xacro:arg name="initial_positions_file" default="initial_positions.yaml" />
     <xacro:arg name="sim" default="real" />
     <!-- Import ada urdf file -->
-    <xacro:include filename="$(find ada_description)/urdf/ada.xacro" />
+    <xacro:include filename="$(find ada_description)/urdf/argallab_jaco.xacro" />
     <!-- Import control_xacro -->
-    <xacro:include filename="ada.ros2_control.xacro" />
-    <xacro:ada_ros2_control name="ADAHardware"
+    <xacro:include filename="argallab_jaco.ros2_control.xacro" />
+    <xacro:argallab_jaco_ros2_control name="JacoHardware"
         initial_positions_file="$(arg initial_positions_file)"
         sim="$(arg sim)" />
